File: hardware/sesam_v2.brd (EAGLE design)
At the start: 70 x 70 mm, 13 parts, among them IC1 337T

Commit message: switched to the correct regulator
Parts:
- removed IC1: 337T, linear:TO220H
- added VREG1: LF33CV, mp_vreg:TO220
- moved C1 2.23 mm to (47.5, 53.3)
Connections:
- net 3V3: now also VREG1.3; no longer IC1.3
- net GND: now also U1.GPIO15, VREG1.2; no longer IC1.1
- net GPIO15: no longer GPIO.3, U1.GPIO15
- net GPIO16: now also GPIO.3
- net POWER: now also VREG1.1; no longer IC1.2
Routing:
- net GPIO16: track 0.00 -> 39.7 mm, vias 0 -> 1
- net GPIO15: track 88.4 -> 57.5 mm, vias 1 -> 0
- net GND: track 15.0 -> 0.00 mm
- net N$7: track 0.00 -> 9.59 mm
- net 3V3: track 144.1 -> 149.1 mm
- net N$8: track 0.00 -> 2.74 mm
- net N$6: track 0.00 -> 2.65 mm
- net POWER: track 9.82 -> 8.97 mm

Commit message: minor tweaks of the board and change of display text size
Routing:
- net GND: track 0.00 -> 15.0 mm
- net N$7: track 9.59 -> 0.00 mm
- net N$8: track 2.74 -> 0.00 mm
- net N$6: track 2.65 -> 0.00 mm
- net GPIO0: track 50.4 -> 51.7 mm
- net GPIO13: track 54.7 -> 53.6 mm
- net 3V3: track 149.1 -> 150.1 mm
- net GPIO12: track 45.8 -> 45.1 mm
- net N$14: track 63.3 -> 62.7 mm
